File: pcb/projects/battery-protection/BatteryProtection.sch (EAGLE design)
At the start: 14 parts, among them U1 BQ29700DSET

Commit message: v1.1 update
Updates to the flight computer:
* update to max31856 tc to digital to support k/j type tc as well as 7
other types
* add pins for iridium sbd message ready and iridium actively
transmitting
* add capacity sense header
* add through hole connection for battery
* remove rs232 level converter - all pins are 5v tolerant on teensy 3.5
and the iridium operates from 3.5-5.5v DC so no need for it
* add imu orientation silk screen as well as arduino pin map silk on
back
* more meaningful LED names
* added end-to-end activation and battery protection schematic

Other updates
* documentation tex file is now local
* add battery protection schematic, board and gerbers as well as renders
Parts:
- removed H1, H4: MOUNT-HOLE2.8, holes:MOUNT-HOLE2.8
Changed lines of the file:
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@@
 <setting verticaltext="up"/>
 </settings>
-<grid distance="0.1" unitdist="inch" unit="inch" style="lines" multiple="1" display="no" altdistance="0.05" altunitdist="inch" altunit="inch"/>
+<grid distance="0.1" unitdist="inch" unit="inch" style="lines" multiple="1" display="no" altdistance="0.01" altunitdist="inch" altunit="inch"/>
 <layers>
 <layer number="1" name="Top" color="4" fill="1" visible="no" active="no"/>
@@
 <part name="FET2" library="KRUPS" deviceset="CSD16406Q3" device=""/>
 <part name="FET1" library="KRUPS" deviceset="CSD16406Q3" device=""/>
-<part name="H1" library="holes" library_urn="urn:adsk.eagle:library:237" deviceset="MOUNT-HOLE" device="2.8" package3d_urn="urn:adsk.eagle:package:14271/1"/>
 <part name="H2" library="holes" library_urn="urn:adsk.eagle:library:237" deviceset="MOUNT-HOLE" device="2.8" package3d_urn="urn:adsk.eagle:package:14271/1"/>
 <part name="H3" library="holes" library_urn="urn:adsk.eagle:library:237" deviceset="MOUNT-HOLE" device="2.8" package3d_urn="urn:adsk.eagle:package:14271/1"/>
-<part name="H4" library="holes" library_urn="urn:adsk.eagle:library:237" deviceset="MOUNT-HOLE" device="2.8" package3d_urn="urn:adsk.eagle:package:14271/1"/>
 <part name="CELL+" library="holes" library_urn="urn:adsk.eagle:library:237" deviceset="MOUNT-PAD-ROUND" device="2.8" package3d_urn="urn:adsk.eagle:package:14281/1"/>
 <part name="CELL-" library="holes" library_urn="urn:adsk.eagle:library:237" deviceset="MOUNT-PAD-ROUND" device="2.8" package3d_urn="urn:adsk.eagle:package:14281/1"/>
@@
 <attribute name="VALUE" x="96.2406" y="92.4814" size="2.0828" layer="96" ratio="6" rot="SMR180"/>
 </instance>
-<instance part="H1" gate="G$1" x="27.94" y="58.42" smashed="yes">
-<attribute name="NAME" x="29.972" y="59.0042" size="1.778" layer="95"/>
-<attribute name="VALUE" x="29.972" y="55.9562" size="1.778" layer="96"/>
-</instance>
 <instance part="H2" gate="G$1" x="27.94" y="48.26" smashed="yes">
 <attribute name="NAME" x="29.972" y="48.8442" size="1.778" layer="95"/>
@@
 <attribute name="VALUE" x="57.912" y="55.9562" size="1.778" layer="96"/>
 </instance>
-<instance part="H4" gate="G$1" x="55.88" y="48.26" smashed="yes">
-<attribute name="NAME" x="57.912" y="48.8442" size="1.778" layer="95"/>
-<attribute name="VALUE" x="57.912" y="45.7962" size="1.778" layer="96"/>
-</instance>
 <instance part="CELL+" gate="G$1" x="170.18" y="139.7" smashed="yes">
