File: pcb/projects/kreme-iss/kreme-iss.brd (EAGLE design)
At the start: 101.6 x 60.6 mm, 89 parts, among them IC1 ADG609RU, IC3 ADG609RU, P1 53048-0810, P2 53048-0810, U1 MCP73831/OT, U10 MAX31855KASA+T21-0041B_8-M, U11 MAX31855KASA+T21-0041B_8-M, U2 LP2985IM5-1.8/NOPB, U3 COM-13909, U4 ADXL377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

Commit message: v1.1 update
Updates to the flight computer:
* update to max31856 tc to digital to support k/j type tc as well as 7
other types
* add pins for iridium sbd message ready and iridium actively
transmitting
* add capacity sense header
* add through hole connection for battery
* remove rs232 level converter - all pins are 5v tolerant on teensy 3.5
and the iridium operates from 3.5-5.5v DC so no need for it
* add imu orientation silk screen as well as arduino pin map silk on
back
* more meaningful LED names
* added end-to-end activation and battery protection schematic

Other updates
* documentation tex file is now local
* add battery protection schematic, board and gerbers as well as renders
Parts:
- removed C12, C7: 0.1uF, adafruit:C0603
- removed C13: 0.01uF, adafruit:C0603
- removed LED6, LED7, LED8: (no value), adafruit:CHIP-LED0603
- removed R12, R16, R17: 470, rcl:R0603
- removed U$34: MAX3232E, TI_radio:SSOP-16
- removed U10, U11: MAX31855KASA+T21-0041B_8-M, max31855:21-0041B_8-M
- added CAPSENSE: 53048-0810, con-molex-picoblade:53048-0810
- added U12, U13: MAX31856MUD+, MAX31856:SOP65P640X110-14N
- added VBAT_PTH: (no value), pinhead:1X02
- moved C5 30.0 mm to (85.3, 24.9), turned to 0 degrees
- moved C6 28.6 mm to (79.0, 22.9), turned to 90 degrees
- moved C32 8.45 mm to (71.6, 24.9), turned to 0 degrees
- moved LED1 6.14 mm to (13.7, 6.86), turned to 270 degrees
- moved LED2 5.71 mm to (18.0, 6.86), turned to 90 degrees
- moved R11 3.84 mm to (35.6, 6.86)
- moved R4 3.78 mm to (13.7, 8.89), turned to 180 degrees
- moved LED3 3.21 mm to (25.7, 6.86), turned to 90 degrees
- moved LED4 3.05 mm to (30.5, 6.86), turned to 90 degrees
- moved R9 2.75 mm to (25.7, 8.64)
- moved R10 2.74 mm to (30.5, 8.64)
- moved R8 2.62 mm to (18.0, 8.89)
- moved LED5 1.80 mm to (35.6, 5.08), turned to 90 degrees
- moved CHARGE 0.80 mm to (9.78, 32.4)
- moved R1 0.76 mm to (22.9, 46.2), turned to 90 degrees
- renumbered POWER_SW to ACTIVATION_SW
Connections:
- removed net LED6: R12.1, U$1.8
- removed net LED7: R16.1, U$1.24
- removed net LED8: R17.1, U$1.25
- removed net N$10: C6.2, U$34.3
- removed net N$11: C5.1, U$34.4
- removed net N$14: C13.1, U$34.6
- removed net N$17: C7.2, U$34.2
- removed net N$29: LED6.A, R12.2
- removed net N$30: LED7.A, R16.2
- removed net N$31: LED8.A, R17.2
- removed net N$5: C5.2, U$34.5
- removed net N$8: C6.1, U$34.1
- removed net R232: U$34.8, X3.P$2
- removed net T232: U$34.7, X3.P$1
- new net CAPSENSE0: CAPSENSE.4, U$1.0/RX
- new net CAPSENSE1: CAPSENSE.2, U$1.1/TX
- new net CAPSENSE2: CAPSENSE.6, U$1.15/A1
- new net CAPSENSE3: CAPSENSE.8, U$1.30
- new net IRIDIUM_STATUS: U$1.A22/DAC1, X3.P$5
- new net IRIDIUM_TX_ACT: U$1.21/DAC0, X3.P$6
- net 3V3: now also C5.1, C6.1, U12.5, U12.8, U13.5, U13.8; no longer C12.1, U$34.16, U10.4, U11.4
- net CS@TC1: now also U13.9; no longer U10.6
- net CS@TC2: now also U12.9; no longer U11.6
- net GND: now also C5.2, C6.2, CAPSENSE.1, CAPSENSE.3, CAPSENSE.5, CAPSENSE.7, U12.1, U12.14, U13.1, U13.14, VBAT_PTH.1, X3.P$2; no longer C12.2, C13.2, C7.1, LED6.C, LED7.C, LED8.C, U$34.15, U10.1, U11.1, X3.P$5, X3.P$6
- net MISO: now also U12.11, U13.11; no longer U10.7, U11.7
- net MOSI: now also U12.12, U13.12
- net RIRI: now also X3.P$4; no longer U$34.9
- net SCLK: now also U12.10, U13.10; no longer U10.5, U11.5
- net TIRI: now also X3.P$3; no longer U$34.10
- net TM_MUX1: now also U13.2, U13.3; no longer U10.2
- net TM_MUX2: now also U12.2, U12.3; no longer U11.2
- net TP_MUX1: now also U13.4; no longer U10.3
- net TP_MUX2: now also U12.4; no longer U11.3
- net V+_IRIDIUM: now also X3.P$1; no longer X3.P$3, X3.P$4
- net VBAT: now also VBAT_PTH.2
Routing:
- net CAPSENSE0: track 0.00 -> 48.1 mm
- net TIRI: track 26.0 -> 68.6 mm
- net CAPSENSE1: track 0.00 -> 41.6 mm
- net T232: track 40.9 -> 0.00 mm
- net IRIDIUM_STATUS: track 0.00 -> 39.0 mm, vias 0 -> 1
- net RIRI: track 26.8 -> 65.0 mm
- net R232: track 36.7 -> 0.00 mm
- net MOSI: track 57.3 -> 93.2 mm, vias 2 -> 5
- net IRIDIUM_TX_ACT: track 0.00 -> 34.9 mm, vias 0 -> 1
- net CAPSENSE2: track 0.00 -> 30.7 mm, vias 0 -> 1
- net 3V3: track 239.7 -> 258.1 mm, vias 9 -> 8
- net ACT: track 41.8 -> 58.7 mm
- net V+_IRIDIUM: track 22.1 -> 8.66 mm
- net CAPSENSE3: track 0.00 -> 10.5 mm
- net LED6: track 8.35 -> 0.00 mm
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Other:
- board text added: "+X"
- board text added: "+Y"
- board text added: "+Z"
- board text added: "0 CAPSENSE0 1 CAPSENSE1 3 LED1 (IR_ON) 4 LED2 (IR_SIG) 5 LED3 (IR_TX) 6 LED4 (ISM_TX) 7 LED5 (ACT) 9 CS_ISM"
- board text added: "11 MOSI 12 MISO 13 SCLK 14 BAT_STAT 15 CAPSENSE2 16 MUX0 17 MUX1 18 SDA 19 SCL"
- board text added: "20 CS@TC1 21 CS@TC2 A8 BAT_SENSE 23 ACT (IRIDIUM ON/OFF) 28 RESET_ISM 28 INT_ISM 30 CAPSENSE3 31 RIRI (IRIDIUM OUTPUT) 32 TIRI (IRIDIUM INPUT) 33 RADIO_OFF_SIG"
- board text added: "34 FSYNC (IMU) 35 INT (IMU) 36 XOUT (A17) 37 YOUT (A18) 38 ZOUT (A19) A21 IRIDIUM_TX_ACT A22 IRIDIUM_STATUS"
- board text added: "5v only"
- board text added: "ACT"
- board text added: "Arduino Pin"
- board text added: "Cap.Ch.0"
- board text added: "Cap.Ch.1"
- board text added: "Cap.Ch.2"
- board text added: "Cap.Ch.3"
- board text added: "IR_ON"
- board text added: "IR_SIG"
- board text added: "IR_TX"
- board text added: "ISM_TX"
- board text added: "KREPE Flight Computer V1.1 University of Kentucky 2020"
- board text added: "Net Name"
- board text added: "ST"
- board text removed: "KREPE Flight Computer V1 University of Kentucky 2020"
