File: pcb/projects/flight-computer/flight-computer.sch (EAGLE design)
At the start: 95 parts, among them CN1 4U#20329, IC1 ADG609RU, IC2 ATSAMD21E, IC3 ADG609RU, P1 53048-0810, P2 53048-0810, U1 MCP73831/OT, U10 SN74LVC1G08DCKR, U11 DPS310XTSA1, U12 MAX31856MUD+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

Commit message: add document revision
Other:
- note added: "12/15/20"
- note added: "12/15/2020"
- note added: "6.1"
- note added: "KFC-6.1"
- note added: "KREPE Flight Computer"
- note added: "LiIon Charging + Monitoring"
- note removed: "6.0"
- note removed: "KRUPS Main Board"
- note removed: "LiPo Charging + Monitoring"
Changed lines of the file:
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@@
 <wire x1="147.32" y1="45.72" x2="147.32" y2="35.56" width="0.254" layer="94" style="longdash"/>
 <text x="96.52" y="38.1" size="5.08" layer="94">Mounting Holes</text>
-<text x="162.56" y="17.78" size="2.54" layer="94">KRUPS Main Board</text>
-<text x="238.76" y="7.62" size="2.54" layer="94">6.0</text>
+<text x="162.56" y="17.78" size="2.54" layer="94">KREPE Flight Computer</text>
+<text x="238.76" y="7.62" size="2.54" layer="94">6.1</text>
+<text x="162.56" y="7.62" size="2.54" layer="94">KFC-6.1</text>
+<text x="162.56" y="1.524" size="2.54" layer="94">12/15/2020</text>
 </plain>
 <instances>
@@
 <wire x1="147.32" y1="104.14" x2="0" y2="104.14" width="0.254" layer="94" style="longdash"/>
 <wire x1="248.92" y1="96.52" x2="248.92" y2="83.82" width="0.254" layer="94" style="longdash"/>
-<text x="162.56" y="17.78" size="2.54" layer="94">KRUPS Main Board</text>
-<text x="238.76" y="7.62" size="2.54" layer="94">6.0</text>
+<text x="238.76" y="7.62" size="2.54" layer="94">6.1</text>
+<text x="162.56" y="7.62" size="2.54" layer="94">KFC-6.1</text>
+<text x="162.814" y="1.27" size="2.54" layer="94">12/15/2020</text>
+<text x="162.56" y="17.78" size="2.54" layer="94">KREPE Flight Computer</text>
 </plain>
 <instances>
@@
 <instance part="FRAME2" gate="G$1" x="0" y="0" smashed="yes"/>
 <instance part="FRAME2" gate="G$2" x="147.32" y="0" smashed="yes">
-<attribute name="LAST_DATE_TIME" x="160.02" y="1.27" size="2.54" layer="94"/>
 <attribute name="SHEET" x="233.68" y="1.27" size="2.54" layer="94"/>
 </instance>
@@
 <text x="13.97" y="176.784" size="5.08" layer="94">Charge Control</text>
 <text x="87.63" y="176.276" size="5.08" layer="94">Power Headers</text>
-<text x="30.48" y="78.74" size="5.08" layer="94">LiPo Charging + Monitoring</text>
+<text x="30.48" y="78.74" size="5.08" layer="94">LiIon Charging + Monitoring</text>
 <wire x1="248.92" y1="124.46" x2="248.92" y2="114.3" width="0.254" layer="94" style="longdash"/>
 <text x="172.72" y="175.26" size="5.08" layer="94">1.8V Regulator</text>
-<text x="162.56" y="17.78" size="2.54" layer="94">KRUPS Main Board</text>
-<text x="238.76" y="7.62" size="2.54" layer="94">6.0</text>
+<text x="238.76" y="7.62" size="2.54" layer="94">6.1</text>
+<text x="162.56" y="7.62" size="2.54" layer="94">KFC-6.1</text>
+<text x="162.814" y="1.27" size="2.54" layer="94">12/15/20</text>
+<text x="162.56" y="17.78" size="2.54" layer="94">KREPE Flight Computer</text>
 </plain>
 <instances>
@@
 <instance part="FRAME3" gate="G$1" x="0" y="0" smashed="yes"/>
 <instance part="FRAME3" gate="G$2" x="147.32" y="0" smashed="yes">
-<attribute name="LAST_DATE_TIME" x="160.02" y="1.27" size="2.54" layer="94"/>
 <attribute name="SHEET" x="233.68" y="1.27" size="2.54" layer="94"/>
 </instance>
@@
 <wire x1="147.32" y1="175.26" x2="248.92" y2="175.26" width="0.254" layer="94" style="longdash"/>
 <text x="180.34" y="119.38" size="5.08" layer="94">ISM Radio</text>
-<text x="162.56" y="17.78" size="2.54" layer="94">KRUPS Main Board</text>
-<text x="238.76" y="7.62" size="2.54" layer="94">6.0</text>
+<text x="238.76" y="7.62" size="2.54" layer="94">6.1</text>
 <wire x1="147.32" y1="175.26" x2="0" y2="175.26" width="0.254" layer="94" style="longdash"/>
 <text x="35.56" y="177.8" size="5.08" layer="94">Status LEDs</text>
@@
 <wire x1="248.92" y1="114.3" x2="147.32" y2="114.3" width="0.254" layer="94" style="longdash"/>
 <text x="154.94" y="177.8" size="5.08" layer="94">Barometric Pressure Sensor</text>
+<text x="162.56" y="7.62" size="2.54" layer="94">KFC-6.1</text>
+<text x="162.56" y="17.78" size="2.54" layer="94">KREPE Flight Computer</text>
 </plain>
 <instances>
@@
 <text x="119.38" y="137.16" size="2.032" layer="94">https://cdn-learn.adafruit.com/assets/assets/000/049/778/original/adafruit_products_Adafruit_Trinket_M0.png?1514756138
 https://github.com/adafruit/Adafruit-Trinket-M0-PCB</text>
+<text x="190.5" y="7.62" size="2.54" layer="94">KFC-6.1</text>
+<text x="190.5" y="17.78" size="2.54" layer="94">KREPE Flight Computer</text>
+<text x="190.246" y="1.778" size="2.54" layer="94">12/15/20</text>
+<text x="264.16" y="7.62" size="2.54" layer="94">6.1</text>
 </plain>
 <instances>
@@
 <instance part="FRAME5" gate="G$1" x="0" y="0" smashed="yes"/>
 <instance part="FRAME5" gate="G$2" x="172.72" y="0" smashed="yes">
-<attribute name="LAST_DATE_TIME" x="185.42" y="1.27" size="2.54" layer="94"/>
 <attribute name="SHEET" x="259.08" y="1.27" size="2.54" layer="94"/>
-<attribute name="DRAWING_NAME" x="190.5" y="19.05" size="2.54" layer="94"/>
 </instance>
 <instance part="JP1" gate="A" x="152.4" y="45.72" smashed="yes">
