File: pcb/projects/flight-computer-v2/main_board.brd (EAGLE design)
At the start: 127 x 64.4 mm, 110 parts, among them J1 B4B-PH-K-S(LF)(SN), J2 B4B-PH-K-S(LF)(SN), J3 B4B-PH-K-S(LF)(SN), J4 B4B-PH-K-S(LF)(SN), J5 B4B-PH-K-S(LF)(SN), J6 B4B-PH-K-S(LF)(SN), J7 104031-0811, J8 B4B-PH-K-S(LF)(SN), J9 U.FL-R-SMT(10), U1 COM-13909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

Commit message: updates to layout
Parts:
- removed C16: 0.01uF, rcl:C0603
- removed C2, C3, C4, C5: 0.1uF, rcl:C0603
- removed R1, R3, R4: 100k, microbuilder:0603-NO
- removed U$3: IRF7313PBF, COM-13909:SO-8
- removed U$34: MAX3232E, TI_radio:SSOP-16
- added JP2: (no value), pinhead:1X04
- added SJ10, SJ11, SJ8: (no value), jumper:SJ_2
- moved J9 131.3 mm to (64.8, 59.7), turned to 90 degrees
- moved SJ1 31.8 mm to (24.1, 53.3), turned to 0 degrees
- moved SJ2 28.1 mm to (24.1, 57.1), turned to 180 degrees
- moved U$1 22.2 mm to (14.0, 59.7), turned to 90 degrees
- moved R2 19.6 mm to (17.1, 56.4), turned to 270 degrees
- moved SJ3 19.1 mm to (76.2, 36.3), turned to 180 degrees
- moved C7 17.7 mm to (35.6, 52.1), turned to 270 degrees
- moved J2 16.6 mm to (36.8, 62.2)
- moved J4 15.3 mm to (22.9, 62.2)
- moved C6 13.5 mm to (35.6, 57.1), turned to 270 degrees
- moved U$2 13.0 mm to (31.8, 52.1), turned to 270 degrees
- moved SJ7 12.8 mm to (85.1, 38.1)
- moved R6 11.5 mm to (20.3, 15.2), turned to 180 degrees
- moved C29 11.4 mm to (44.5, 50.8), turned to 270 degrees
- moved R5 10.2 mm to (26.7, 15.2)
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Connections:
- removed net 3.3V: C4.1, U$34.16
- removed net EN: JP3.2, R45.2, U13.3
- removed net GATE_GPS: JP3.9, R4.1, U$3.2
- removed net GND_CONVERTERS: U$1.7, U$1.8
- removed net GND_GPS: J2.4, U$3.7, U$3.8
- removed net GND_RADIO: U$3.5, U$3.6, U1.1, U1.10, U1.8
- removed net N$1: R5.2, R6.2
- removed net N$10: C2.2, U$34.3
- removed net N$17: C5.2, U$34.5
- removed net N$18: C16.1, U$34.6
- removed net N$19: C3.1, U$34.2
- removed net SCL1: U10.19, U4.19, U5.19, U7.19, U8.19, U9.19
- removed net SDA1: U10.20, U4.20, U5.20, U7.20, U8.20, U9.20
- new net 3V32_CTRL: JP3.9, R45.2, U13.3
- net 3V3: now also SJ8.1; no longer C7.2, U$2.16
- net 3V32: now also SJ8.3
- net 5V: now also JP2.4, SJ10.3, SJ11.3; no longer J2.3, J4.3
- net GATE_IRIDIUM: no longer R1.1
- net GATE_PI: now also R5.1, U$5.2; no longer R6.1, U$5.4
- net GATE_RADIO: no longer R3.1, U$3.4
- net GATE_SPEC: now also R6.1, U$5.4; no longer R5.1, U$5.2
- net GND: now also JP2.1, R2.2, R5.2, R6.2, U1.1, U1.10, U1.8; no longer C16.2, C3.2, C4.2, C9.1, U$2.15, U$3.1, U$3.3, U$34.15
- net GND_IRIDIUM: now also C9.1, J2.4, U$1.7, U$1.8, U$2.15
- net GND_PI: now also U$5.7, U$5.8; no longer U$5.5, U$5.6
- net GND_SPEC: now also U$5.5, U$5.6; no longer U$5.7, U$5.8
- net N$16: now also J4.3, SJ11.2; no longer C5.1, U$34.4
- net N$6: now also J2.3, SJ10.2; no longer R1.2, R2.2, R3.2, R4.2
- net N$9: now also C7.2, SJ8.2, U$2.16; no longer C2.1, U$34.1
- net R232: no longer U$34.8
- net R232_GPS: no longer U$34.13
- net RGPS: no longer U$34.12
- net RIRI: no longer U$34.9
- net SCL: now also U10.19, U4.19, U5.19, U7.19, U8.19, U9.19
- net SDA: now also U10.20, U4.20, U5.20, U7.20, U8.20, U9.20
- net T232: no longer U$34.7
- net T232_GPS: no longer U$34.14
- net TGPS: no longer U$34.11
- net TIRI: no longer U$34.10
- net VBAT: now also JP2.3
- net VIN: now also JP2.2, SJ10.1, SJ11.1
Routing:
- net 3V3: track 0.00 -> 250.1 mm, vias 0 -> 5
- net 5V: track 0.00 -> 123.6 mm, vias 0 -> 1
- net SCK: track 0.00 -> 89.9 mm, vias 0 -> 1
- net MOSI: track 0.00 -> 78.4 mm
- net MISO: track 0.00 -> 69.7 mm
- net RADIO_SS: track 0.00 -> 59.2 mm
- net RADIO_RESET: track 0.00 -> 56.4 mm
- net VBAT: track 0.00 -> 55.7 mm, vias 0 -> 1
- net TGPS: track 0.00 -> 51.0 mm
- net RGPS: track 0.00 -> 42.2 mm
- net GND: track 0.00 -> 40.5 mm, vias 0 -> 24
- net 3V32: track 0.00 -> 38.0 mm
- net GATE_SPEC: track 0.00 -> 35.3 mm, vias 0 -> 1
- net N$6: track 0.00 -> 31.8 mm, vias 0 -> 2
- net SD_CS: track 0.00 -> 26.0 mm
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- added copper zone on layer 1, net GND
- added copper zone on layer 16, net GND
- added copper zone on layer 1, net GND_IRIDIUM
- added copper zone on layer 1, net GND_PI
- added copper zone on layer 1, net GND_SPEC

Commit message: update PCB and libraries
Parts:
- added JP4: (no value), pinhead:1X02
- added R1, R9: 10k, rcl:R0603
- added R3: 7.5k, rcl:R0603
- added R4: 4.3k, rcl:R0603
- added SJ9: (no value), jumper:SJ
- moved C26 29.6 mm to (95.4, 15.0), turned to 270 degrees
- moved C28 26.7 mm to (109.2, 15.2), turned to 270 degrees
- moved C23 23.4 mm to (108.0, 41.9), turned to 180 degrees
- moved J3 23.3 mm to (50.8, 24.1), turned to 90 degrees
- moved SJ3 17.2 mm to (88.6, 24.5)
- moved C24 13.0 mm to (86.4, 45.7), turned to 270 degrees
- moved R32 12.7 mm to (104.1, 24.1)
- moved C19 12.7 mm to (101.6, 30.5)
- moved R8 11.7 mm to (39.4, 43.2)
- moved R7 10.9 mm to (39.4, 44.5)
- moved SJ7 9.18 mm to (87.4, 29.2)
- moved R25 6.48 mm to (97.8, 15.2), turned to 90 degrees
- moved C25 3.61 mm to (100.1, 47.6), turned to 90 degrees
- moved R39 3.60 mm to (112.9, 48.4)
- moved R40 3.59 mm to (110.5, 48.3)
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- renumbered U$1 to U12, U$2 to U11, U$5 to U14
Connections:
- removed net GND_I2C: J3.4
- new net N$1: JP4.1, SJ9.1, U1.13
- new net N$10: R1.2, R3.2, U8.16
- new net N$17: R4.2, R9.2, U7.16
- net 3V3: now also R1.1, R9.1, U6.12; no longer U8.16
- net 3V32: now also JP4.2, SJ9.2; no longer U1.13
- net GND: now also C9.1, J3.4, R3.1, R4.1, U11.15, U6.7; no longer U7.16
- net GND_IRIDIUM: no longer C9.1, U11.15
- net N$3: now also SJ2.2; no longer SJ1.2
- net N$4: now also SJ1.2; no longer SJ2.2
- net SCL: now also U6.13
- net SDA: now also U6.14
Routing:
- net SDA: track 0.00 -> 208.4 mm, vias 0 -> 9
- net 3V3: track 250.1 -> 441.0 mm, vias 5 -> 13
- net SCL: track 0.00 -> 190.1 mm, vias 0 -> 9
- net GND: track 40.5 -> 149.6 mm, vias 24 -> 85
- net GATE_PI: track 3.97 -> 29.3 mm, vias 0 -> 1
- net GATE_IRIDIUM: track 6.13 -> 29.5 mm, vias 0 -> 1
- net 3V32_CTRL: track 2.99 -> 24.0 mm, vias 0 -> 1
- net N$44: track 4.95 -> 22.6 mm
- net N$58: track 0.00 -> 11.3 mm
- net N$1: track 0.00 -> 9.10 mm
- net N$10: track 0.00 -> 8.10 mm
- net N$62: track 0.00 -> 7.32 mm
- net N$57: track 0.00 -> 7.25 mm
- net N$60: track 0.00 -> 7.21 mm
- net N$34: track 0.00 -> 6.90 mm
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Other:
- board text added: "+"
- board text added: "-"
- board text added: "3V"
- board text added: "3V3 GND"
- board text added: "5v"
- board text added: "915Mhz ANT"
- board text added: "ADDR SELECT"
- board text added: "ADDR SELECT FxS300"
- board text added: "GND"
- board text added: "GND 5V TX RX"
- board text added: "GND 5V or VIN R232 T232"
- board text added: "GND VIN GND 5V"
- board text added: "GND VIN VBAT 5V"
- board text added: "I2C"
- board text added: "J2"
- board text added: "J4"
- board text added: "KREPE-2 Flight Computer"
- board text added: "Matt Ruffner, Evan Wells, Kirsten Ford, Bruno Tacci, Dr. Alexandre Martin Dr. Bill Smith Dr. Savio Poovathingal"
- board text added: "POL Switch 3.3V TTL Serial"
- board text added: "POL Switch RS232 Serial"
- board text added: "Radio power"
- board text added: "SCL SDA 3V3 GND"
- board text added: "TC1"
- board text added: "TC2"
- board text added: "TC3"
- board text added: "TC4"
- board text added: "TC5"
- board text added: "U11 source"
- board text added: "V SELECT"
- board text added: "VIN"
- board text added: "VIN GND VBAT GND"
- board text added: "ext."
- board text added: "feat."
